Commit message: docs: add kinematics info

File: rbda_description/robots/rbda.urdf (robot description, URDF)
Before this commit: robot rbda, 18 links, 17 joints
Joints:
- removed joint joint4
- removed joint joint5
- added joint joint_4: type continuous, parent link_3, child link_4, origin xyz=0.0 0.0 0.0 rpy=0.0 0.0 0.0, axis 0 1 0
- added joint joint_5: type continuous, parent link_4, child link_5, origin xyz=0.0 -0.00645 0.28600 rpy=0.0 0.0 0.0, axis 0 1 0

Commit message: docs: fix inertia of links

File: rbda_description/robots/rbda.urdf (robot description, URDF)
Before this commit: robot rbda, 18 links, 17 joints
Joints:
- joint joint_13: origin xyz=0.0 0.0 -0.005 rpy=0.0 0.0 0.0 -> xyz=0.0 0.0 0.0 rpy=0.0 0.0 0.0
- joint joint_14: origin xyz=0.0 0.0 0.34900 rpy=0.0 0.0 0.0 -> xyz=0.0 0.0 0.34400 rpy=0.0 0.0 0.0
- joint joint_6: origin xyz=0.0 0.0 -0.005 rpy=0.0 0.0 0.0 -> xyz=0.0 0.0 0.0 rpy=0.0 0.0 0.0
- joint joint_7: origin xyz=0.0 0.0 0.34900 rpy=0.0 0.0 0.0 -> xyz=0.0 0.0 0.34400 rpy=0.0 0.0 0.0
